File: _autosave-pcb-guide.kicad_sch (KiCad schematic)
At the start: 24 parts, among them J1 USB_B_Mini, SW1 SW_Push, U1 ATmega32U4-A, Y1 16MHz

Commit message: Add submodules
Parts:
- SW1: footprint random-keyboard-parts:SKQG-1155865 -> Button_Switch_THT:SW_PUSH_6mm
Changed lines of the file:
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@@
     (property "Reference" "SW1" (id 0) (at 104.14 45.72 0))
     (property "Value" "SW_Push" (id 1) (at 104.14 48.26 0))
-    (property "Footprint" "random-keyboard-parts:SKQG-1155865" (id 2) (at 104.14 48.26 0)
+    (property "Footprint" "Button_Switch_THT:SW_PUSH_6mm" (id 2) (at 104.14 48.26 0)
       (effects (font (size 1.27 1.27)) hide)
     )
@@
     )
     (path "/f5248ab6-7069-45ad-b798-c8f1a0a0e3a6"
-      (reference "SW1") (unit 1) (value "SW_Push") (footprint "random-keyboard-parts:SKQG-1155865")
+      (reference "SW1") (unit 1) (value "SW_Push") (footprint "Button_Switch_THT:SW_PUSH_6mm")
     )
     (path "/543e8d72-6b60-4cb9-b68c-88731afec46b"
